Commit message: Give the 3D model real link bulk: 10 mm hips, 30 mm thighs, pointed shins, and a 30 mm chassis.
Co-authored-by: Cursor <cursoragent@cursor.com>

File: hexapod_description/urdf/body.urdf (robot description, URDF)
Before this commit: robot hexapod_body, 7 links, 6 joints
Links:
- link base_link: geometry visual box size=0.146564 0.186859 0.030

File: hexapod_description/urdf/hexapod.urdf (robot description, URDF)
Before this commit: robot hexapod, 43 links, 42 joints
Links:
- link LF_coxa: geometry visual box size=0.053 0.010 0.010
- link LF_femur: geometry visual box size=0.07736 0.030 0.030
- link LF_shin1: geometry visual box size=0.022358 0.008 0.064
- link LF_shin2: geometry visual box size=0.071518 0.006 0.037
- link LF_shin3: geometry visual box size=0.03114 0.004 0.009
- link LM_coxa: geometry visual box size=0.053 0.010 0.010
- link LM_femur: geometry visual box size=0.07736 0.030 0.030
- link LM_shin1: geometry visual box size=0.022358 0.008 0.064
- link LM_shin2: geometry visual box size=0.071518 0.006 0.037
- link LM_shin3: geometry visual box size=0.03114 0.004 0.009
- link LR_coxa: geometry visual box size=0.053 0.010 0.010
- link LR_femur: geometry visual box size=0.07736 0.030 0.030
- link LR_shin1: geometry visual box size=0.022358 0.008 0.064
- link LR_shin2: geometry visual box size=0.071518 0.006 0.037
- link LR_shin3: geometry visual box size=0.03114 0.004 0.009
- link RF_coxa: geometry visual box size=0.053 0.010 0.010
- link RF_femur: geometry visual box size=0.07736 0.030 0.030
- link RF_shin1: geometry visual box size=0.022358 0.008 0.064
- link RF_shin2: geometry visual box size=0.071518 0.006 0.037
- link RF_shin3: geometry visual box size=0.03114 0.004 0.009
- link RM_coxa: geometry visual box size=0.053 0.010 0.010
- link RM_femur: geometry visual box size=0.07736 0.030 0.030
- link RM_shin1: geometry visual box size=0.022358 0.008 0.064
- link RM_shin2: geometry visual box size=0.071518 0.006 0.037
- link RM_shin3: geometry visual box size=0.03114 0.004 0.009
- link RR_coxa: geometry visual box size=0.053 0.010 0.010
- link RR_femur: geometry visual box size=0.07736 0.030 0.030
- link RR_shin1: geometry visual box size=0.022358 0.008 0.064
- link RR_shin2: geometry visual box size=0.071518 0.006 0.037
- link RR_shin3: geometry visual box size=0.03114 0.004 0.009
- link base_link: geometry visual box size=0.146564 0.186859 0.030

File: hexapod_description/urdf/leg_one.urdf (robot description, URDF)
Before this commit: robot hexapod_leg, 7 links, 6 joints
Links:
- link coxa_link: geometry visual box size=0.053 0.010 0.010
- link femur_link: geometry visual box size=0.07736 0.030 0.030
- link shin1_link: geometry visual box size=0.022358 0.008 0.064
- link shin2_link: geometry visual box size=0.071518 0.006 0.037
- link shin3_link: geometry visual box size=0.03114 0.004 0.009
